File: connectors.kicad_sch (KiCad schematic)
At the start: 4 parts, among them J1 Conn_01x36, J2 Conn_01x18, J5 Conn_01x17, J6 Conn_01x03

Commit message: Add h-bridges for magnetorquers
Parts:
- added J3: Conn_01x06, symbol Connector_Generic:Conn_01x06
- added J4: Conn_01x02, symbol Connector_Generic:Conn_01x02
- added J7: Conn_01x09, symbol Connector_Generic:Conn_01x09
Connections:
- new net MCTRL1_1: J7.1 (Pin_1)
- new net MCTRL1_2: J7.2 (Pin_2)
- new net MCTRL2_1: J7.4 (Pin_4)
- new net MCTRL2_2: J7.5 (Pin_5)
- new net MCTRL3_1: J7.7 (Pin_7)
- new net MCTRL3_2: J7.8 (Pin_8)
- new net MSLEEP1: J7.3 (Pin_3)
- new net MSLEEP2: J7.6 (Pin_6)
- new net MSLEEP3: J7.9 (Pin_9)
- new net MTQ1+: J3.1 (Pin_1)
- new net MTQ1-: J3.2 (Pin_2)
- new net MTQ2+: J3.3 (Pin_3)
- new net MTQ2-: J3.4 (Pin_4)
- new net MTQ3+: J3.5 (Pin_5)
- new net MTQ3-: J3.6 (Pin_6)
Other:
- note added: "from EPS"
- note added: "magnetorquer in (from compute board)"
- note added: "to magnetorquers"
